Commit message: updates

File: robots/urdf/panda_limb_repo/panda_limb_repo.urdf (robot description, URDF)
Before this commit: robot panda, 12 links, 11 joints
Joints:
- joint panda_joint3: axis (none) -> 0.0 0.0 1.0; type fixed -> continuous

File: robots/urdf/panda_limb_repo/panda_limb_repo_with_limits.urdf (robot description, URDF)
Before this commit: robot panda, 12 links, 11 joints
Joints:
- joint panda_joint3: axis (none) -> 0.0 0.0 1.0; type fixed -> continuous

Commit message: fix fixed horizon implementation

File: robots/urdf/panda_limb_repo/panda_limb_repo.urdf (robot description, URDF)
Before this commit: robot panda, 12 links, 11 joints
Joints:
- joint panda_joint3: axis 0.0 0.0 1.0 -> (none); type continuous -> fixed

File: robots/urdf/panda_limb_repo/panda_limb_repo_with_limits.urdf (robot description, URDF)
Before this commit: robot panda, 12 links, 11 joints
Joints:
- joint panda_joint3: axis 0.0 0.0 1.0 -> (none); type continuous -> fixed
